File: PCB design files/hackercard.kicad_sch (KiCad schematic)
At the start: 5 parts, among them U1 NT3H2111W0FHKH

Commit message: Replace C2295 with C84256
Parts:
- LED1: JLC Part # C2295 -> C84256
Changed lines of the file:
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@@
 			)
 		)
-		(property "JLC Part #" "C2295"
+		(property "JLC Part #" "C84256"
 			(at 68.58 87.63 0)
 			(hide yes)
